Commit message: Update scene to work with the scene_parser

File: benchmark_suite/config/bbt_primitive_scene.urdf.xacro (robot description, xacro)
@@ -3,38 +3,35 @@
   <xacro:include filename="$(find scene_parser)/config/utils.xacro" />
   <xacro:include filename="$(find scene_parser)/config/opencrate.urdf.xacro" />
+  <!-- Used to get bb information from real meshes -->
+  <xacro:include filename="$(find moveit_benchmark_suite_resources)/objects/geometry.xacro" />
   <link name="world" />
-  <xacro:property name="cube_dimensions" value="0.0254 0.0254 0.0254" />
-  <xacro:property name="cube_name" value="cube" />
-  <xacro:property name="dl" value="_" />
-  <xacro:opencrate name="clear_box1"
+  <xacro:framebox name="boxlid"
+                  frame_id="world"
+                  dimensions="${boxlid['bby']} ${boxlid['bbz']} ${boxlid['bbx']}"
+                  xyz="${0.16 + boxlid['bby']/2} 0 0"/>
+  <xacro:opencrate name="clearbox1"
                    frame_id="world"
-                   xyz="${0.429/2 + 0.16} ${0.292/2 + 0.01/2} 0"
-                   dimensions="0.429 0.292 0.149"
-                   thickness="0.01"/>
-  <xacro:opencrate name="clear_box2"
-                   frame_id="clear_box1"
-                   xyz="0 ${-0.292-0.01} 0"
-                   dimensions="0.429 0.292 0.149"
-                   thickness="0.01"/>
-  <xacro:framebox name="box_lid1"
-                  frame_id="clear_box1"
-                  dimensions="0.429 0.01 0.292"
-                  xyz="0 ${-0.292/2 - 0.01/2} ${0.292/2}" />
-  <xacro:subframe name="clear_box2"
-                  subframe="bottom"
-                  xyz="0 0 0.01" />
-  <!-- TODO add to utility file -->
-  <xacro:macro name="linearpattern" params="current:=0 frame_id:=^ index:=0 max:=^ xyz:=^ gap:=^">
+                   xyz="${0.16 + clearbox['bby']/2} ${-(clearbox['bbx']/2 + boxlid['bbz']/2)} 0" rpy="0 0 0"
+                   dimensions="${clearbox['bby']} ${clearbox['bbx']} ${clearbox['bbz']}"
+                   thickness="0.00709"/>
+  <xacro:opencrate name="clearbox2"
+                   frame_id="clearbox1"
+                   xyz="0 ${clearbox['bbx'] + boxlid['bbz']} 0" rpy="0 0 0"
+                   dimensions="${clearbox['bby']} ${clearbox['bbx']} ${clearbox['bbz']}"
+                   thickness="0.00709"/>
+  <xacro:macro name="linearpattern" params="current:=0 frame_id:=^ index:=0 max:=^ xyz:=^ rpy=^|'0 0 0' gap:=^">
     <xacro:if value="${max > current}">
-      <xacro:framebox name="wood_block${index+current}"
+      <xacro:framebox name="woodblock${index+current}"
                       frame_id="${frame_id}"
-                      dimensions="0.0254 0.0254 0.0254"
-                      xyz="${float(xyz.split()[0]) + current*float(gap.split()[0])} ${float(xyz.split()[1]) + current*float(gap.split()[1])} ${float(xyz.split()[2]) + current*float(gap.split()[2])}" />
+                      dimensions="${woodblock['bbx']} ${woodblock['bby']} ${woodblock['bbz']}"
+                      xyz="${float(xyz.split()[0]) + current*float(gap.split()[0])}
+                           ${float(xyz.split()[1]) + current*float(gap.split()[1])}
+                           ${float(xyz.split()[2]) + current*float(gap.split()[2])}" />
       <xacro:linearpattern current="${current+1}" index="${index}"/>
     </xacro:if>
   </xacro:macro>
-  <xacro:linearpattern index="1"  max="4"  frame_id="clear_box2/bottom" gap="0 ${0.0254*2} 0" xyz="${3*0.0254} ${(-3*0.0254)} ${0.0254/2}"/>
-  <xacro:linearpattern index="5"  max="4"  frame_id="wood_block1" gap="0 ${0.0254*2} 0" xyz="${-2*0.0254} 0 0"/>
-  <xacro:linearpattern index="9"  max="4"  frame_id="wood_block5" gap="0 ${0.0254*2} 0" xyz="${-2*0.0254} 0 0"/>
-  <xacro:linearpattern index="13" max="4"  frame_id="wood_block9" gap="0 ${0.0254*2} 0" xyz="${-2*0.0254} 0 0"/>
+  <xacro:linearpattern index="1"  max="4"  frame_id="clearbox1"  gap="0 ${woodblock['bby']*2} 0" xyz="${3*woodblock['bbx']} ${(-3*woodblock['bbx'])} 0" rpy="0 0 0"/>
+  <xacro:linearpattern index="5"  max="4"  frame_id="woodblock1/bottom" gap="0 ${woodblock['bby']*2} 0" xyz="${-2*woodblock['bbx']} 0 0"/>
+  <xacro:linearpattern index="9"  max="4"  frame_id="woodblock5/bottom" gap="0 ${woodblock['bby']*2} 0" xyz="${-2*woodblock['bbx']} 0 0"/>
+  <xacro:linearpattern index="13" max="4"  frame_id="woodblock9/bottom" gap="0 ${woodblock['bby']*2} 0" xyz="${-2*woodblock['bbx']} 0 0"/>
 </robot>
