Commit message: fix typo breaking mtc scene

File: resources/objects/metadata.xacro (robot description, xacro)
@@ -10,5 +10,5 @@
   <xacro:property name="mug"        value="${load_yaml(pkg_path + 'mug.yaml')['mug']}"/>
   <xacro:property name="plate"      value="${load_yaml(pkg_path + 'plate.yaml')['plate']}"/>
-  <xacro:property name="soupecan"   value="${load_yaml(pkg_path + 'soupecan.yaml')['soupecan']}"/>
+  <xacro:property name="soupcan"   value="${load_yaml(pkg_path + 'soupcan.yaml')['soupcan']}"/>
   <xacro:property name="woodblock"  value="${load_yaml(pkg_path + 'woodblock.yaml')['woodblock']}"/>
 </robot>

Commit message: Fix xacro deprecated warning in Noetic

File: resources/objects/metadata.xacro (robot description, xacro)
@@ -3,12 +3,12 @@
   <xacro:property name="pkg_path"   value="$(find moveit_benchmark_suite_resources)/objects/"/>
   <!-- Load metadata of all meshes -->
-  <xacro:property name="apcshelf"   value="${load_yaml(pkg_path + 'apcshelf.yaml')['apcshelf']}"/>
-  <xacro:property name="bowl"       value="${load_yaml(pkg_path + 'bowl.yaml')['bowl']}"/>
-  <xacro:property name="boxlid"     value="${load_yaml(pkg_path + 'boxlid.yaml')['boxlid']}"/>
-  <xacro:property name="clearbox"   value="${load_yaml(pkg_path + 'clearbox.yaml')['clearbox']}"/>
-  <xacro:property name="drill"      value="${load_yaml(pkg_path + 'drill.yaml')['drill']}"/>
-  <xacro:property name="mug"        value="${load_yaml(pkg_path + 'mug.yaml')['mug']}"/>
-  <xacro:property name="plate"      value="${load_yaml(pkg_path + 'plate.yaml')['plate']}"/>
-  <xacro:property name="soupcan"   value="${load_yaml(pkg_path + 'soupcan.yaml')['soupcan']}"/>
-  <xacro:property name="woodblock"  value="${load_yaml(pkg_path + 'woodblock.yaml')['woodblock']}"/>
+  <xacro:property name="apcshelf"   value="${xacro.load_yaml(pkg_path + 'apcshelf.yaml')['apcshelf']}"/>
+  <xacro:property name="bowl"       value="${xacro.load_yaml(pkg_path + 'bowl.yaml')['bowl']}"/>
+  <xacro:property name="boxlid"     value="${xacro.load_yaml(pkg_path + 'boxlid.yaml')['boxlid']}"/>
+  <xacro:property name="clearbox"   value="${xacro.load_yaml(pkg_path + 'clearbox.yaml')['clearbox']}"/>
+  <xacro:property name="drill"      value="${xacro.load_yaml(pkg_path + 'drill.yaml')['drill']}"/>
+  <xacro:property name="mug"        value="${xacro.load_yaml(pkg_path + 'mug.yaml')['mug']}"/>
+  <xacro:property name="plate"      value="${xacro.load_yaml(pkg_path + 'plate.yaml')['plate']}"/>
+  <xacro:property name="soupcan"    value="${xacro.load_yaml(pkg_path + 'soupcan.yaml')['soupcan']}"/>
+  <xacro:property name="woodblock"  value="${xacro.load_yaml(pkg_path + 'woodblock.yaml')['woodblock']}"/>
 </robot>

Commit message: Add unit box mesh from blender

File: resources/objects/metadata.xacro (robot description, xacro)
@@ -3,12 +3,13 @@
   <xacro:property name="pkg_path"   value="$(find moveit_benchmark_suite_resources)/objects/"/>
   <!-- Load metadata of all meshes -->
-  <xacro:property name="apcshelf"   value="${xacro.load_yaml(pkg_path + 'apcshelf.yaml')['apcshelf']}"/>
-  <xacro:property name="bowl"       value="${xacro.load_yaml(pkg_path + 'bowl.yaml')['bowl']}"/>
-  <xacro:property name="boxlid"     value="${xacro.load_yaml(pkg_path + 'boxlid.yaml')['boxlid']}"/>
-  <xacro:property name="clearbox"   value="${xacro.load_yaml(pkg_path + 'clearbox.yaml')['clearbox']}"/>
-  <xacro:property name="drill"      value="${xacro.load_yaml(pkg_path + 'drill.yaml')['drill']}"/>
-  <xacro:property name="mug"        value="${xacro.load_yaml(pkg_path + 'mug.yaml')['mug']}"/>
-  <xacro:property name="plate"      value="${xacro.load_yaml(pkg_path + 'plate.yaml')['plate']}"/>
-  <xacro:property name="soupcan"    value="${xacro.load_yaml(pkg_path + 'soupcan.yaml')['soupcan']}"/>
-  <xacro:property name="woodblock"  value="${xacro.load_yaml(pkg_path + 'woodblock.yaml')['woodblock']}"/>
+  <xacro:property name="apcshelf"           value="${xacro.load_yaml(pkg_path + 'apcshelf.yaml')['apcshelf']}"/>
+  <xacro:property name="bowl"               value="${xacro.load_yaml(pkg_path + 'bowl.yaml')['bowl']}"/>
+  <xacro:property name="boxlid"             value="${xacro.load_yaml(pkg_path + 'boxlid.yaml')['boxlid']}"/>
+  <xacro:property name="clearbox"           value="${xacro.load_yaml(pkg_path + 'clearbox.yaml')['clearbox']}"/>
+  <xacro:property name="drill"              value="${xacro.load_yaml(pkg_path + 'drill.yaml')['drill']}"/>
+  <xacro:property name="mug"                value="${xacro.load_yaml(pkg_path + 'mug.yaml')['mug']}"/>
+  <xacro:property name="plate"              value="${xacro.load_yaml(pkg_path + 'plate.yaml')['plate']}"/>
+  <xacro:property name="soupcan"            value="${xacro.load_yaml(pkg_path + 'soupcan.yaml')['soupcan']}"/>
+  <xacro:property name="unit_box_blender"   value="${xacro.load_yaml(pkg_path + 'unit_box_blender.yaml')['unit_box_blender']}"/>
+  <xacro:property name="woodblock"          value="${xacro.load_yaml(pkg_path + 'woodblock.yaml')['woodblock']}"/>
 </robot>

Commit message: Add unit box mesh from solidworks

File: resources/objects/metadata.xacro (robot description, xacro)
@@ -3,13 +3,14 @@
   <xacro:property name="pkg_path"   value="$(find moveit_benchmark_suite_resources)/objects/"/>
   <!-- Load metadata of all meshes -->
-  <xacro:property name="apcshelf"           value="${xacro.load_yaml(pkg_path + 'apcshelf.yaml')['apcshelf']}"/>
-  <xacro:property name="bowl"               value="${xacro.load_yaml(pkg_path + 'bowl.yaml')['bowl']}"/>
-  <xacro:property name="boxlid"             value="${xacro.load_yaml(pkg_path + 'boxlid.yaml')['boxlid']}"/>
-  <xacro:property name="clearbox"           value="${xacro.load_yaml(pkg_path + 'clearbox.yaml')['clearbox']}"/>
-  <xacro:property name="drill"              value="${xacro.load_yaml(pkg_path + 'drill.yaml')['drill']}"/>
-  <xacro:property name="mug"                value="${xacro.load_yaml(pkg_path + 'mug.yaml')['mug']}"/>
-  <xacro:property name="plate"              value="${xacro.load_yaml(pkg_path + 'plate.yaml')['plate']}"/>
-  <xacro:property name="soupcan"            value="${xacro.load_yaml(pkg_path + 'soupcan.yaml')['soupcan']}"/>
-  <xacro:property name="unit_box_blender"   value="${xacro.load_yaml(pkg_path + 'unit_box_blender.yaml')['unit_box_blender']}"/>
-  <xacro:property name="woodblock"          value="${xacro.load_yaml(pkg_path + 'woodblock.yaml')['woodblock']}"/>
+  <xacro:property name="apcshelf"             value="${xacro.load_yaml(pkg_path + 'apcshelf.yaml')['apcshelf']}"/>
+  <xacro:property name="bowl"                 value="${xacro.load_yaml(pkg_path + 'bowl.yaml')['bowl']}"/>
+  <xacro:property name="boxlid"               value="${xacro.load_yaml(pkg_path + 'boxlid.yaml')['boxlid']}"/>
+  <xacro:property name="clearbox"             value="${xacro.load_yaml(pkg_path + 'clearbox.yaml')['clearbox']}"/>
+  <xacro:property name="drill"                value="${xacro.load_yaml(pkg_path + 'drill.yaml')['drill']}"/>
+  <xacro:property name="mug"                  value="${xacro.load_yaml(pkg_path + 'mug.yaml')['mug']}"/>
+  <xacro:property name="plate"                value="${xacro.load_yaml(pkg_path + 'plate.yaml')['plate']}"/>
+  <xacro:property name="soupcan"              value="${xacro.load_yaml(pkg_path + 'soupcan.yaml')['soupcan']}"/>
+  <xacro:property name="unit_box_blender"     value="${xacro.load_yaml(pkg_path + 'unit_box_blender.yaml')['unit_box_blender']}"/>
+  <xacro:property name="unit_box_solidworks"  value="${xacro.load_yaml(pkg_path + 'unit_box_solidworks.yaml')['unit_box_solidworks']}"/>
+  <xacro:property name="woodblock"            value="${xacro.load_yaml(pkg_path + 'woodblock.yaml')['woodblock']}"/>
 </robot>
