Commit message: Add clearbox subframe for adding objects in it
Scenes have been changed to use this information.

File: resources/db/bbt/panda/scene_mesh_hq.urdf.xacro (robot description, xacro)
@@ -28,5 +28,6 @@
     </xacro:if>
   </xacro:macro>
-  <xacro:linearpattern index="1"  max="4"  frame_id="clearbox1"  gap="${woodblock['bby']*2} 0 0" xyz="${-3*woodblock['bbx']} ${(-3*woodblock['bbx'])} ${0.00709}" rpy="0 0 ${-pi/2}"/>
+  <xacro:property name="stack_z" value="${clearbox['subframes']['stack']['xyz'][2]}"/>
+  <xacro:linearpattern index="1"  max="4"  frame_id="clearbox1"  gap="${woodblock['bby']*2} 0 0" xyz="${-3*woodblock['bbx']} ${(-3*woodblock['bbx'])} ${stack_z}" rpy="0 0 ${-pi/2}"/>
   <xacro:linearpattern index="5"  max="4"  frame_id="woodblock1" gap="0 ${woodblock['bby']*2} 0" xyz="${-2*woodblock['bbx']} 0 0"/>
   <xacro:linearpattern index="9"  max="4"  frame_id="woodblock5" gap="0 ${woodblock['bby']*2} 0" xyz="${-2*woodblock['bbx']} 0 0"/>

File: resources/db/bbt/panda/scene_primitive.urdf.xacro (robot description, xacro)
@@ -14,5 +14,5 @@
                    xyz="${0.16 + clearbox['bby']/2} ${-(clearbox['bbx']/2 + boxlid['bbz']/2)} 0" rpy="0 0 0"
                    dimensions="${clearbox['bby']} ${clearbox['bbx']} ${clearbox['bbz']}"
-                   thickness="0.00709"/>
+                   thickness="${clearbox['subframes']['stack']['xyz'][2]}"/>
   <xacro:opencrate name="clearbox2"
                    frame_id="clearbox1"

File: resources/objects/geometry.xacro (robot description, xacro)
@@ -34,5 +34,8 @@
                                            stack = dict(  xyz=[0, 0, 0.00624]),
                                            ))}"/>
-  <xacro:property name="clearbox"   value="${dict(bbx=0.284112, bby=0.409485, bbz=0.141286)}"/>
+  <xacro:property name="clearbox"   value="${dict(bbx=0.284112, bby=0.409485, bbz=0.141286,
+                                           subframes=dict(
+                                           stack = dict( xyz=[0, 0, 0.00709]),
+                                           ))}"/>
   <xacro:property name="mug"        value="${dict(bbx=0.11699, bby=0.093089, bbz=0.141286)}"/>
   <xacro:property name="plate"      value="${dict(bbx=0.26015, bby=0.261102, bbz=0.026723,

Commit message: Refactored object metadata

File: resources/db/bbt/panda/scene_mesh_hq.urdf.xacro (robot description, xacro)
@@ -2,18 +2,18 @@
 <robot name="scene" xmlns:xacro="http://www.ros.org/wiki/xacro">
   <xacro:include filename="$(find scene_parser)/config/utils.xacro" />
-  <xacro:include filename="$(find moveit_benchmark_suite_resources)/objects/geometry.xacro" />
+  <xacro:include filename="$(find moveit_benchmark_suite_resources)/objects/metadata.xacro" />
   <link name="world" />
   <xacro:framemesh name="boxlid"
                        frame_id="world"
-                       xyz="${0.16 + boxlid['bby']/2} ${-boxlid['bbz']/2} ${boxlid['bbx']/2}" rpy="0 ${pi/2} ${pi/2}"
-                       resource="package://moveit_benchmark_suite_resources/objects/boxlid_19k.stl"/>
+                       xyz="${0.16 + boxlid['bb'][1]/2} ${-boxlid['bb'][2]/2} ${boxlid['bb'][0]/2}" rpy="0 ${pi/2} ${pi/2}"
+                       metadata="${boxlid}"/>
   <xacro:framemesh name="clearbox1"
                        frame_id="world"
-                       xyz="${0.16 + clearbox['bby']/2} ${-(clearbox['bbx']/2 + boxlid['bbz']/2)} 0" rpy="0 0 ${pi/2}"
-                       resource="package://moveit_benchmark_suite_resources/objects/clearbox_50k.stl"/>
+                       xyz="${0.16 + clearbox['bb'][1]/2} ${-(clearbox['bb'][0]/2 + boxlid['bb'][2]/2)} 0" rpy="0 0 ${pi/2}"
+                       metadata="${clearbox}"/>
   <xacro:framemesh name="clearbox2"
                        frame_id="clearbox1"
-                       xyz="${clearbox['bbx'] + boxlid['bbz']} 0 0" rpy="0 0 0"
-                       resource="package://moveit_benchmark_suite_resources/objects/clearbox_50k.stl"/>
+                       xyz="${clearbox['bb'][0] + boxlid['bb'][2]} 0 0" rpy="0 0 0"
+                       metadata="${clearbox}"/>
   <xacro:macro name="linearpattern" params="current:=0 frame_id:=^ index:=0 max:=^ xyz:=^ rpy=^|'0 0 0' gap:=^">
     <xacro:if value="${max > current}">
@@ -24,12 +24,12 @@
                             ${float(xyz.split()[2]) + current*float(gap.split()[2])}"
                        rpy="${rpy}"
-                       resource="package://moveit_benchmark_suite_resources/objects/woodblock_16k.stl"/>
+                       metadata="${woodblock}"/>
       <xacro:linearpattern current="${current+1}" index="${index}"/>
     </xacro:if>
   </xacro:macro>
   <xacro:property name="stack_z" value="${clearbox['subframes']['stack']['xyz'][2]}"/>
-  <xacro:linearpattern index="1"  max="4"  frame_id="clearbox1"  gap="${woodblock['bby']*2} 0 0" xyz="${-3*woodblock['bbx']} ${(-3*woodblock['bbx'])} ${stack_z}" rpy="0 0 ${-pi/2}"/>
-  <xacro:linearpattern index="5"  max="4"  frame_id="woodblock1" gap="0 ${woodblock['bby']*2} 0" xyz="${-2*woodblock['bbx']} 0 0"/>
-  <xacro:linearpattern index="9"  max="4"  frame_id="woodblock5" gap="0 ${woodblock['bby']*2} 0" xyz="${-2*woodblock['bbx']} 0 0"/>
-  <xacro:linearpattern index="13" max="4"  frame_id="woodblock9" gap="0 ${woodblock['bby']*2} 0" xyz="${-2*woodblock['bbx']} 0 0"/>
+  <xacro:linearpattern index="1"  max="4"  frame_id="clearbox1"  gap="${woodblock['bb'][1]*2} 0 0" xyz="${-3*woodblock['bb'][0]} ${(-3*woodblock['bb'][0])} ${stack_z}" rpy="0 0 ${-pi/2}"/>
+  <xacro:linearpattern index="5"  max="4"  frame_id="woodblock1" gap="0 ${woodblock['bb'][1]*2} 0" xyz="${-2*woodblock['bb'][0]} 0 0"/>
+  <xacro:linearpattern index="9"  max="4"  frame_id="woodblock5" gap="0 ${woodblock['bb'][1]*2} 0" xyz="${-2*woodblock['bb'][0]} 0 0"/>
+  <xacro:linearpattern index="13" max="4"  frame_id="woodblock9" gap="0 ${woodblock['bb'][1]*2} 0" xyz="${-2*woodblock['bb'][0]} 0 0"/>
 </robot>

File: resources/db/bbt/panda/scene_primitive.urdf.xacro (robot description, xacro)
@@ -3,20 +3,19 @@
   <xacro:include filename="$(find scene_parser)/config/utils.xacro" />
   <xacro:include filename="$(find scene_parser)/config/opencrate.urdf.xacro" />
-  <!-- Used to get bb information from real meshes -->
-  <xacro:include filename="$(find moveit_benchmark_suite_resources)/objects/geometry.xacro" />
+  <xacro:include filename="$(find moveit_benchmark_suite_resources)/objects/metadata.xacro" />
   <link name="world" />
   <xacro:framebox name="boxlid"
                   frame_id="world"
-                  dimensions="${boxlid['bby']} ${boxlid['bbz']} ${boxlid['bbx']}"
-                  xyz="${0.16 + boxlid['bby']/2} 0 0"/>
+                  dimensions="${boxlid['bb'][1]} ${boxlid['bb'][2]} ${boxlid['bb'][0]}"
+                  xyz="${0.16 + boxlid['bb'][1]/2} 0 0"/>
   <xacro:opencrate name="clearbox1"
                    frame_id="world"
-                   xyz="${0.16 + clearbox['bby']/2} ${-(clearbox['bbx']/2 + boxlid['bbz']/2)} 0" rpy="0 0 0"
-                   dimensions="${clearbox['bby']} ${clearbox['bbx']} ${clearbox['bbz']}"
+                   xyz="${0.16 + clearbox['bb'][1]/2} ${-(clearbox['bb'][0]/2 + boxlid['bb'][2]/2)} 0" rpy="0 0 0"
+                   dimensions="${clearbox['bb'][1]} ${clearbox['bb'][0]} ${clearbox['bb'][2]}"
                    thickness="${clearbox['subframes']['stack']['xyz'][2]}"/>
   <xacro:opencrate name="clearbox2"
                    frame_id="clearbox1"
-                   xyz="0 ${clearbox['bbx'] + boxlid['bbz']} 0" rpy="0 0 0"
-                   dimensions="${clearbox['bby']} ${clearbox['bbx']} ${clearbox['bbz']}"
+                   xyz="0 ${clearbox['bb'][0] + boxlid['bb'][2]} 0" rpy="0 0 0"
+                   dimensions="${clearbox['bb'][1]} ${clearbox['bb'][0]} ${clearbox['bb'][2]}"
                    thickness="0.00709"/>
   <xacro:macro name="linearpattern" params="current:=0 frame_id:=^ index:=0 max:=^ xyz:=^ rpy=^|'0 0 0' gap:=^">
@@ -24,5 +23,5 @@
       <xacro:framebox name="woodblock${index+current}"
                       frame_id="${frame_id}"
-                      dimensions="${woodblock['bbx']} ${woodblock['bby']} ${woodblock['bbz']}"
+                      dimensions="${woodblock['bb'][0]} ${woodblock['bb'][1]} ${woodblock['bb'][2]}"
                       xyz="${float(xyz.split()[0]) + current*float(gap.split()[0])}
                            ${float(xyz.split()[1]) + current*float(gap.split()[1])}
@@ -31,7 +30,7 @@
     </xacro:if>
   </xacro:macro>
-  <xacro:linearpattern index="1"  max="4"  frame_id="clearbox1"  gap="0 ${woodblock['bby']*2} 0" xyz="${3*woodblock['bbx']} ${(-3*woodblock['bbx'])} 0" rpy="0 0 0"/>
-  <xacro:linearpattern index="5"  max="4"  frame_id="woodblock1/bottom" gap="0 ${woodblock['bby']*2} 0" xyz="${-2*woodblock['bbx']} 0 0"/>
-  <xacro:linearpattern index="9"  max="4"  frame_id="woodblock5/bottom" gap="0 ${woodblock['bby']*2} 0" xyz="${-2*woodblock['bbx']} 0 0"/>
-  <xacro:linearpattern index="13" max="4"  frame_id="woodblock9/bottom" gap="0 ${woodblock['bby']*2} 0" xyz="${-2*woodblock['bbx']} 0 0"/>
+  <xacro:linearpattern index="1"  max="4"  frame_id="clearbox1"  gap="0 ${woodblock['bb'][1]*2} 0" xyz="${3*woodblock['bb'][0]} ${(-3*woodblock['bb'][0])} 0" rpy="0 0 0"/>
+  <xacro:linearpattern index="5"  max="4"  frame_id="woodblock1/bottom" gap="0 ${woodblock['bb'][1]*2} 0" xyz="${-2*woodblock['bb'][0]} 0 0"/>
+  <xacro:linearpattern index="9"  max="4"  frame_id="woodblock5/bottom" gap="0 ${woodblock['bb'][1]*2} 0" xyz="${-2*woodblock['bb'][0]} 0 0"/>
+  <xacro:linearpattern index="13" max="4"  frame_id="woodblock9/bottom" gap="0 ${woodblock['bb'][1]*2} 0" xyz="${-2*woodblock['bb'][0]} 0 0"/>
 </robot>

File: resources/db/openshelf/panda/scene_mesh_hq.urdf.xacro (robot description, xacro)
@@ -3,5 +3,5 @@
   <xacro:include filename="$(find scene_parser)/config/utils.xacro" />
   <xacro:include filename="$(find scene_parser)/config/shelf.urdf.xacro" />
-  <xacro:include filename="$(find moveit_benchmark_suite_resources)/objects/geometry.xacro" />
+  <xacro:include filename="$(find moveit_benchmark_suite_resources)/objects/metadata.xacro" />
   <link name="world" />
   <!-- Create default shelf -->
@@ -18,31 +18,20 @@
                        frame_id="shelf_board1"
                        xyz="0 0 0" rpy="0 0 0"
-                       resource="package://moveit_benchmark_suite_resources/objects/mug_16k.stl"/>
+                       metadata="${mug}"/>
   <xacro:framemesh name="bowl"
                        frame_id="shelf_board2"
                        xyz="0 0 0" rpy="0 0 0"
-                       resource="package://moveit_benchmark_suite_resources/objects/bowl_16k.stl"/>
+                       metadata="${bowl}"/>
   <xacro:framemesh name="plate"
                        frame_id="shelf_board8"
                        xyz="0 0 0" rpy="0 0 0"
-                       resource="package://moveit_benchmark_suite_resources/objects/plate_16k.stl"/>
+                       metadata="${plate}"/>
   <xacro:framemesh name="soupcan"
                        frame_id="shelf_board7"
                        xyz="0.1 0 0" rpy="0 0 0"
-                       resource="package://moveit_benchmark_suite_resources/objects/soupcan_16k.stl"/>
+                       metadata="${soupcan}"/>
   <xacro:framemesh name="drill"
                        frame_id="shelf_board8"
                        xyz="0 0 0" rpy="0 0 0"
-                       resource="package://moveit_benchmark_suite_resources/objects/drill_16k.stl"/>
-  <!-- <xacro:macro name="shelf" params="name -->
-  <!--                                   frame_id -->
-  <!--                                   xyz:='0 0 0' -->
-  <!--                                   rpy:='0 0 0' -->
-  <!--                                   dimensions:='0.6 1.5 1.25' -->
-  <!--                                   h_boards:=5 -->
-  <!--                                   v_boards:=3 -->
-  <!--                                   h_board_thickness:=0.02 -->
-  <!--                                   v_board_thickness:=0.02 -->
-  <!--                                   back_board:=false -->
-  <!--                                   dl:=_"> -->
+                       metadata="${drill}"/>
 </robot>

Commit message: resources: do not override `max`
Reduces these warnings:
> redefining global symbol: max

File: resources/db/bbt/panda/scene_mesh_hq.urdf.xacro (robot description, xacro)
@@ -16,6 +16,6 @@
                        xyz="${clearbox['bb'][0] + boxlid['bb'][2]} 0 0" rpy="0 0 0"
                        metadata="${clearbox}"/>
-  <xacro:macro name="linearpattern" params="current:=0 frame_id:=^ index:=0 max:=^ xyz:=^ rpy=^|'0 0 0' gap:=^">
-    <xacro:if value="${max > current}">
+  <xacro:macro name="linearpattern" params="current:=0 frame_id:=^ index:=0 until:=^ xyz:=^ rpy=^|'0 0 0' gap:=^">
+    <xacro:if value="${until > current}">
       <xacro:framemesh name="woodblock${current+index}"
                        frame_id="${frame_id}"
@@ -29,7 +29,7 @@
   </xacro:macro>
   <xacro:property name="stack_z" value="${clearbox['subframes']['stack']['xyz'][2]}"/>
-  <xacro:linearpattern index="1"  max="4"  frame_id="clearbox1"  gap="${woodblock['bb'][1]*2} 0 0" xyz="${-3*woodblock['bb'][0]} ${(-3*woodblock['bb'][0])} ${stack_z}" rpy="0 0 ${-pi/2}"/>
-  <xacro:linearpattern index="5"  max="4"  frame_id="woodblock1" gap="0 ${woodblock['bb'][1]*2} 0" xyz="${-2*woodblock['bb'][0]} 0 0"/>
-  <xacro:linearpattern index="9"  max="4"  frame_id="woodblock5" gap="0 ${woodblock['bb'][1]*2} 0" xyz="${-2*woodblock['bb'][0]} 0 0"/>
-  <xacro:linearpattern index="13" max="4"  frame_id="woodblock9" gap="0 ${woodblock['bb'][1]*2} 0" xyz="${-2*woodblock['bb'][0]} 0 0"/>
+  <xacro:linearpattern index="1"  until="4"  frame_id="clearbox1"  gap="${woodblock['bb'][1]*2} 0 0" xyz="${-3*woodblock['bb'][0]} ${(-3*woodblock['bb'][0])} ${stack_z}" rpy="0 0 ${-pi/2}"/>
+  <xacro:linearpattern index="5"  until="4"  frame_id="woodblock1" gap="0 ${woodblock['bb'][1]*2} 0" xyz="${-2*woodblock['bb'][0]} 0 0"/>
+  <xacro:linearpattern index="9"  until="4"  frame_id="woodblock5" gap="0 ${woodblock['bb'][1]*2} 0" xyz="${-2*woodblock['bb'][0]} 0 0"/>
+  <xacro:linearpattern index="13" until="4"  frame_id="woodblock9" gap="0 ${woodblock['bb'][1]*2} 0" xyz="${-2*woodblock['bb'][0]} 0 0"/>
 </robot>

File: resources/db/bbt/panda/scene_primitive.urdf.xacro (robot description, xacro)
@@ -19,6 +19,6 @@
                    dimensions="${clearbox['bb'][1]} ${clearbox['bb'][0]} ${clearbox['bb'][2]}"
                    thickness="0.00709"/>
-  <xacro:macro name="linearpattern" params="current:=0 frame_id:=^ index:=0 max:=^ xyz:=^ rpy=^|'0 0 0' gap:=^">
-    <xacro:if value="${max > current}">
+  <xacro:macro name="linearpattern" params="current:=0 frame_id:=^ index:=0 until:=^ xyz:=^ rpy=^|'0 0 0' gap:=^">
+    <xacro:if value="${until > current}">
       <xacro:framebox name="woodblock${index+current}"
                       frame_id="${frame_id}"
@@ -30,7 +30,7 @@
     </xacro:if>
   </xacro:macro>
-  <xacro:linearpattern index="1"  max="4"  frame_id="clearbox1"  gap="0 ${woodblock['bb'][1]*2} 0" xyz="${3*woodblock['bb'][0]} ${(-3*woodblock['bb'][0])} 0" rpy="0 0 0"/>
-  <xacro:linearpattern index="5"  max="4"  frame_id="woodblock1/bottom" gap="0 ${woodblock['bb'][1]*2} 0" xyz="${-2*woodblock['bb'][0]} 0 0"/>
-  <xacro:linearpattern index="9"  max="4"  frame_id="woodblock5/bottom" gap="0 ${woodblock['bb'][1]*2} 0" xyz="${-2*woodblock['bb'][0]} 0 0"/>
-  <xacro:linearpattern index="13" max="4"  frame_id="woodblock9/bottom" gap="0 ${woodblock['bb'][1]*2} 0" xyz="${-2*woodblock['bb'][0]} 0 0"/>
+  <xacro:linearpattern index="1"  until="4"  frame_id="clearbox1"  gap="0 ${woodblock['bb'][1]*2} 0" xyz="${3*woodblock['bb'][0]} ${(-3*woodblock['bb'][0])} 0" rpy="0 0 0"/>
+  <xacro:linearpattern index="5"  until="4"  frame_id="woodblock1/bottom" gap="0 ${woodblock['bb'][1]*2} 0" xyz="${-2*woodblock['bb'][0]} 0 0"/>
+  <xacro:linearpattern index="9"  until="4"  frame_id="woodblock5/bottom" gap="0 ${woodblock['bb'][1]*2} 0" xyz="${-2*woodblock['bb'][0]} 0 0"/>
+  <xacro:linearpattern index="13" until="4"  frame_id="woodblock9/bottom" gap="0 ${woodblock['bb'][1]*2} 0" xyz="${-2*woodblock['bb'][0]} 0 0"/>
 </robot>
