Commit message: Fix package path resolution

File: resources/robots/panda/urdf/panda.urdf (robot description, URDF)
Before this commit: robot panda, 12 links, 11 joints
Links:
- link panda_hand: geometry collision mesh filename=package://moveit_benchmark_suite_resources/robots/panda/mes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; visual mesh filename=package://moveit_benchmark_suite_resources/robots/panda/mes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
- link panda_leftfinger: geometry collision mesh filename=package://moveit_benchmark_suite_resources/robots/panda/mes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; visual mesh filename=package://moveit_benchmark_suite_resources/robots/panda/mes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
- link panda_link0: geometry collision mesh filename=package://moveit_benchmark_suite_resources/robots/panda/mes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; visual mesh filename=package://moveit_benchmark_suite_resources/robots/panda/mes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
- link panda_link1: geometry collision mesh filename=package://moveit_benchmark_suite_resources/robots/panda/mes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; visual mesh filename=package://moveit_benchmark_suite_resources/robots/panda/mes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
- link panda_link2: geometry collision mesh filename=package://moveit_benchmark_suite_resources/robots/panda/mes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; visual mesh filename=package://moveit_benchmark_suite_resources/robots/panda/mes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
- link panda_link3: geometry collision mesh filename=package://moveit_benchmark_suite_resources/robots/panda/mes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; visual mesh filename=package://moveit_benchmark_suite_resources/robots/panda/mes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
- link panda_link4: geometry collision mesh filename=package://moveit_benchmark_suite_resources/robots/panda/mes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; visual mesh filename=package://moveit_benchmark_suite_resources/robots/panda/mes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
- link panda_link5: geometry collision mesh filename=package://moveit_benchmark_suite_resources/robots/panda/mes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; visual mesh filename=package://moveit_benchmark_suite_resources/robots/panda/mes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
- link panda_link6: geometry collision mesh filename=package://moveit_benchmark_suite_resources/robots/panda/mes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; visual mesh filename=package://moveit_benchmark_suite_resources/robots/panda/mes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
- link panda_link7: geometry collision mesh filename=package://moveit_benchmark_suite_resources/robots/panda/mes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; visual mesh filename=package://moveit_benchmark_suite_resources/robots/panda/mes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
- link panda_rightfinger: geometry collision mesh filename=package://moveit_benchmark_suite_resources/robots/panda/mes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; visual mesh filename=package://moveit_benchmark_suite_resources/robots/panda/mes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

File: resources/robots/robotiq/85_gripper/urdf/robotiq_85_gripper.urdf.xacro (robot description, xacro)
@@ -1,5 +1,5 @@
 <?xml version="1.0"?>
 <robot name="robotiq_85_gripper" xmlns:xacro="http://ros.org/wiki/xacro">
-	<xacro:include filename="$(find robowflex_resources)/robotiq/85_gripper/urdf/robotiq_85_gripper.transmission.xacro" />
+	<xacro:include filename="$(find moveit_benchmark_suite_resources/robots)/robotiq/85_gripper/urdf/robotiq_85_gripper.transmission.xacro" />
 	<xacro:property name="pi" value="3.14159"/>
 	<xacro:macro name="mimic_joint_plugin_gazebo" params="name_prefix parent_joint mimic_joint has_pid:=false multiplier:=1.0 offset:=0 sensitiveness:=0.0 max_effort:=1.0 robot_namespace:=''">
@@ -30,10 +30,10 @@
 			<visual>
 				<geometry>
-					<mesh filename="package://robowflex_resources/robotiq/85_gripper/meshes/visual/robotiq_85_base_link.dae"/>
-				</geometry>
-			</visual>
-			<collision>
-				<geometry>
-					<mesh filename="package://robowflex_resources/robotiq/85_gripper/meshes/collision/robotiq_85_base_link.stl"/>
+					<mesh filename="package://moveit_benchmark_suite_resources/robots/robotiq/85_gripper/meshes/visual/robotiq_85_base_link.dae"/>
+				</geometry>
+			</visual>
+			<collision>
+				<geometry>
+					<mesh filename="package://moveit_benchmark_suite_resources/robots/robotiq/85_gripper/meshes/collision/robotiq_85_base_link.stl"/>
 				</geometry>
 			</collision>
@@ -87,10 +87,10 @@
 			<visual>
 				<geometry>
-					<mesh filename="package://robowflex_resources/robotiq/85_gripper/meshes/visual/robotiq_85_knuckle_link.dae"/>
-				</geometry>
-			</visual>
-			<collision>
-				<geometry>
-					<mesh filename="package://robowflex_resources/robotiq/85_gripper/meshes/collision/robotiq_85_knuckle_link.stl"/>
+					<mesh filename="package://moveit_benchmark_suite_resources/robots/robotiq/85_gripper/meshes/visual/robotiq_85_knuckle_link.dae"/>
+				</geometry>
+			</visual>
+			<collision>
+				<geometry>
+					<mesh filename="package://moveit_benchmark_suite_resources/robots/robotiq/85_gripper/meshes/collision/robotiq_85_knuckle_link.stl"/>
 				</geometry>
 			</collision>
@@ -106,10 +106,10 @@
 			<visual>
 				<geometry>
-					<mesh filename="package://robowflex_resources/robotiq/85_gripper/meshes/visual/robotiq_85_knuckle_link.dae"/>
-				</geometry>
-			</visual>
-			<collision>
-				<geometry>
-					<mesh filename="package://robowflex_resources/robotiq/85_gripper/meshes/collision/robotiq_85_knuckle_link.stl"/>
+					<mesh filename="package://moveit_benchmark_suite_resources/robots/robotiq/85_gripper/meshes/visual/robotiq_85_knuckle_link.dae"/>
+				</geometry>
+			</visual>
+			<collision>
+				<geometry>
+					<mesh filename="package://moveit_benchmark_suite_resources/robots/robotiq/85_gripper/meshes/collision/robotiq_85_knuckle_link.stl"/>
 				</geometry>
 			</collision>
@@ -135,10 +135,10 @@
 			<visual>
 				<geometry>
-					<mesh filename="package://robowflex_resources/robotiq/85_gripper/meshes/visual/robotiq_85_finger_link.dae"/>
-				</geometry>
-			</visual>
-			<collision>
-				<geometry>
-					<mesh filename="package://robowflex_resources/robotiq/85_gripper/meshes/collision/robotiq_85_finger_link.stl"/>
+					<mesh filename="package://moveit_benchmark_suite_resources/robots/robotiq/85_gripper/meshes/visual/robotiq_85_finger_link.dae"/>
+				</geometry>
+			</visual>
+			<collision>
+				<geometry>
+					<mesh filename="package://moveit_benchmark_suite_resources/robots/robotiq/85_gripper/meshes/collision/robotiq_85_finger_link.stl"/>
 				</geometry>
 			</collision>
@@ -154,10 +154,10 @@
 			<visual>
 				<geometry>
-					<mesh filename="package://robowflex_resources/robotiq/85_gripper/meshes/visual/robotiq_85_finger_link.dae"/>
-				</geometry>
-			</visual>
-			<collision>
-				<geometry>
-					<mesh filename="package://robowflex_resources/robotiq/85_gripper/meshes/collision/robotiq_85_finger_link.stl"/>
+					<mesh filename="package://moveit_benchmark_suite_resources/robots/robotiq/85_gripper/meshes/visual/robotiq_85_finger_link.dae"/>
+				</geometry>
+			</visual>
+			<collision>
+				<geometry>
+					<mesh filename="package://moveit_benchmark_suite_resources/robots/robotiq/85_gripper/meshes/collision/robotiq_85_finger_link.stl"/>
 				</geometry>
 			</collision>
@@ -195,10 +195,10 @@
 			<visual>
 				<geometry>
-					<mesh filename="package://robowflex_resources/robotiq/85_gripper/meshes/visual/robotiq_85_inner_knuckle_link.dae"/>
-				</geometry>
-			</visual>
-			<collision>
-				<geometry>
-					<mesh filename="package://robowflex_resources/robotiq/85_gripper/meshes/collision/robotiq_85_inner_knuckle_link.stl"/>
+					<mesh filename="package://moveit_benchmark_suite_resources/robots/robotiq/85_gripper/meshes/visual/robotiq_85_inner_knuckle_link.dae"/>
+				</geometry>
+			</visual>
+			<collision>
+				<geometry>
+					<mesh filename="package://moveit_benchmark_suite_resources/robots/robotiq/85_gripper/meshes/collision/robotiq_85_inner_knuckle_link.stl"/>
 				</geometry>
 			</collision>
@@ -214,10 +214,10 @@
 			<visual>
 				<geometry>
-					<mesh filename="package://robowflex_resources/robotiq/85_gripper/meshes/visual/robotiq_85_inner_knuckle_link.dae"/>
-				</geometry>
-			</visual>
-			<collision>
-				<geometry>
-					<mesh filename="package://robowflex_resources/robotiq/85_gripper/meshes/collision/robotiq_85_inner_knuckle_link.stl"/>
+					<mesh filename="package://moveit_benchmark_suite_resources/robots/robotiq/85_gripper/meshes/visual/robotiq_85_inner_knuckle_link.dae"/>
+				</geometry>
+			</visual>
+			<collision>
+				<geometry>
+					<mesh filename="package://moveit_benchmark_suite_resources/robots/robotiq/85_gripper/meshes/collision/robotiq_85_inner_knuckle_link.stl"/>
 				</geometry>
 			</collision>
@@ -255,10 +255,10 @@
 			<visual>
 				<geometry>
-					<mesh filename="package://robowflex_resources/robotiq/85_gripper/meshes/visual/robotiq_85_finger_tip_link.dae"/>
-				</geometry>
-			</visual>
-			<collision>
-				<geometry>
-					<mesh filename="package://robowflex_resources/robotiq/85_gripper/meshes/collision/robotiq_85_finger_tip_link.stl"/>
+					<mesh filename="package://moveit_benchmark_suite_resources/robots/robotiq/85_gripper/meshes/visual/robotiq_85_finger_tip_link.dae"/>
+				</geometry>
+			</visual>
+			<collision>
+				<geometry>
+					<mesh filename="package://moveit_benchmark_suite_resources/robots/robotiq/85_gripper/meshes/collision/robotiq_85_finger_tip_link.stl"/>
 				</geometry>
 			</collision>
@@ -283,10 +283,10 @@
 			<visual>
 				<geometry>
-					<mesh filename="package://robowflex_resources/robotiq/85_gripper/meshes/visual/robotiq_85_finger_tip_link.dae"/>
-				</geometry>
-			</visual>
-			<collision>
-				<geometry>
-					<mesh filename="package://robowflex_resources/robotiq/85_gripper/meshes/collision/robotiq_85_finger_tip_link.stl"/>
+					<mesh filename="package://moveit_benchmark_suite_resources/robots/robotiq/85_gripper/meshes/visual/robotiq_85_finger_tip_link.dae"/>
+				</geometry>
+			</visual>
+			<collision>
+				<geometry>
+					<mesh filename="package://moveit_benchmark_suite_resources/robots/robotiq/85_gripper/meshes/collision/robotiq_85_finger_tip_link.stl"/>
 				</geometry>
 			</collision>

File: resources/robots/robotiq/85_gripper/urdf/robotiq_arg85_description.urdf.xacro (robot description, xacro)
@@ -2,5 +2,5 @@
 <robot
   name="robotiq_85_gripper"  xmlns:xacro="http://ros.org/wiki/xacro">
-  <xacro:include filename="$(find robowflex_resources)/robotiq/85_gripper/urdf/robotiq_85_gripper.transmission.xacro" />
+  <xacro:include filename="$(find moveit_benchmark_suite_resources/robots)/robotiq/85_gripper/urdf/robotiq_85_gripper.transmission.xacro" />
 	<xacro:property name="pi" value="3.14159"/>
   <xacro:macro name="robotiq_85_gripper" params="prefix parent *origin">
@@ -32,19 +32,19 @@
       <geometry>
         <mesh
-          filename="package://robowflex_resources/robotiq/85_gripper/meshes/arg/robotiq_85_base_link_fine.STL" />
-      </geometry>
-      <material
-        name="">
-        <color
-          rgba="0.1 0.1 0.1 1" />
-      </material>
-    </visual>
-    <collision>
-      <origin
-        xyz="0 0 0"
-        rpy="0 0 0" />
-      <geometry>
-        <mesh
-          filename="package://robowflex_resources/robotiq/85_gripper/meshes/arg/robotiq_85_base_link_coarse.STL" />
+          filename="package://moveit_benchmark_suite_resources/robots/robotiq/85_gripper/meshes/arg/robotiq_85_base_link_fine.STL" />
+      </geometry>
+      <material
+        name="">
+        <color
+          rgba="0.1 0.1 0.1 1" />
+      </material>
+    </visual>
+    <collision>
+      <origin
+        xyz="0 0 0"
+        rpy="0 0 0" />
+      <geometry>
+        <mesh
+          filename="package://moveit_benchmark_suite_resources/robots/robotiq/85_gripper/meshes/arg/robotiq_85_base_link_coarse.STL" />
       </geometry>
     </collision>
@@ -90,19 +90,19 @@
       <geometry>
         <mesh
-          filename="package://robowflex_resources/robotiq/85_gripper/meshes/arg/outer_knuckle_fine.STL" />
-      </geometry>
-      <material
-        name="">
-        <color
-          rgba="0.1 0.1 0.1 1" />
-      </material>
-    </visual>
-    <collision>
-      <origin
-        xyz="0 0 0"
-        rpy="0 0 0" />
-      <geometry>
-        <mesh
-          filename="package://robowflex_resources/robotiq/85_gripper/meshes/arg/outer_knuckle_coarse.STL" />
+          filename="package://moveit_benchmark_suite_resources/robots/robotiq/85_gripper/meshes/arg/outer_knuckle_fine.STL" />
+      </geometry>
+      <material
+        name="">
+        <color
+          rgba="0.1 0.1 0.1 1" />
+      </material>
+    </visual>
+    <collision>
+      <origin
+        xyz="0 0 0"
+        rpy="0 0 0" />
+      <geometry>
+        <mesh
+          filename="package://moveit_benchmark_suite_resources/robots/robotiq/85_gripper/meshes/arg/outer_knuckle_coarse.STL" />
       </geometry>
     </collision>
@@ -152,19 +152,19 @@
       <geometry>
         <mesh
-          filename="package://robowflex_resources/robotiq/85_gripper/meshes/arg/outer_finger_fine.STL" />
-      </geometry>
-      <material
-        name="">
-        <color
-          rgba="0.1 0.1 0.1 1" />
-      </material>
-    </visual>
-    <collision>
-      <origin
-        xyz="0 0 0"
-        rpy="0 0 0" />
-      <geometry>
-        <mesh
-          filename="package://robowflex_resources/robotiq/85_gripper/meshes/arg/outer_finger_coarse.STL" />
+          filename="package://moveit_benchmark_suite_resources/robots/robotiq/85_gripper/meshes/arg/outer_finger_fine.STL" />
+      </geometry>
+      <material
+        name="">
+        <color
+          rgba="0.1 0.1 0.1 1" />
+      </material>
+    </visual>
+    <collision>
+      <origin
+        xyz="0 0 0"
+        rpy="0 0 0" />
+      <geometry>
+        <mesh
+          filename="package://moveit_benchmark_suite_resources/robots/robotiq/85_gripper/meshes/arg/outer_finger_coarse.STL" />
       </geometry>
     </collision>
@@ -214,19 +214,19 @@
       <geometry>
         <mesh
-          filename="package://robowflex_resources/robotiq/85_gripper/meshes/arg/inner_knuckle_fine.STL" />
-      </geometry>
-      <material
-        name="">
-        <color
-          rgba="0.1 0.1 0.1 1" />
-      </material>
-    </visual>
-    <collision>
-      <origin
-        xyz="0 0 0"
-        rpy="0 0 0" />
-      <geometry>
-        <mesh
-          filename="package://robowflex_resources/robotiq/85_gripper/meshes/arg/inner_knuckle_coarse.STL" />
+          filename="package://moveit_benchmark_suite_resources/robots/robotiq/85_gripper/meshes/arg/inner_knuckle_fine.STL" />
+      </geometry>
+      <material
+        name="">
+        <color
+          rgba="0.1 0.1 0.1 1" />
+      </material>
+    </visual>
+    <collision>
+      <origin
+        xyz="0 0 0"
+        rpy="0 0 0" />
+      <geometry>
+        <mesh
+          filename="package://moveit_benchmark_suite_resources/robots/robotiq/85_gripper/meshes/arg/inner_knuckle_coarse.STL" />
       </geometry>
     </collision>
@@ -276,19 +276,19 @@
       <geometry>
         <mesh
-          filename="package://robowflex_resources/robotiq/85_gripper/meshes/arg/inner_finger_fine.STL" />
-      </geometry>
-      <material
-        name="">
-        <color
-          rgba="0.1 0.1 0.1 1" />
-      </material>
-    </visual>
-    <collision>
-      <origin
-        xyz="0 0 0"
-        rpy="0 0 0" />
-      <geometry>
-        <mesh
-          filename="package://robowflex_resources/robotiq/85_gripper/meshes/arg/inner_finger_coarse.STL" />
+          filename="package://moveit_benchmark_suite_resources/robots/robotiq/85_gripper/meshes/arg/inner_finger_fine.STL" />
+      </geometry>
+      <material
+        name="">
+        <color
+          rgba="0.1 0.1 0.1 1" />
+      </material>
+    </visual>
+    <collision>
+      <origin
+        xyz="0 0 0"
+        rpy="0 0 0" />
+      <geometry>
+        <mesh
+          filename="package://moveit_benchmark_suite_resources/robots/robotiq/85_gripper/meshes/arg/inner_finger_coarse.STL" />
       </geometry>
     </collision>
@@ -337,19 +337,19 @@
       <geometry>
         <mesh
-          filename="package://robowflex_resources/robotiq/85_gripper/meshes/arg/inner_knuckle_fine.STL" />
-      </geometry>
-      <material
-        name="">
-        <color
-          rgba="0.1 0.1 0.1 1" />
-      </material>
-    </visual>
-    <collision>
-      <origin
-        xyz="0 0 0"
-        rpy="0 0 0" />
-      <geometry>
-        <mesh
-          filename="package://robowflex_resources/robotiq/85_gripper/meshes/arg/inner_knuckle_coarse.STL" />
+          filename="package://moveit_benchmark_suite_resources/robots/robotiq/85_gripper/meshes/arg/inner_knuckle_fine.STL" />
+      </geometry>
+      <material
+        name="">
+        <color
+          rgba="0.1 0.1 0.1 1" />
+      </material>
+    </visual>
+    <collision>
+      <origin
+        xyz="0 0 0"
+        rpy="0 0 0" />
+      <geometry>
+        <mesh
+          filename="package://moveit_benchmark_suite_resources/robots/robotiq/85_gripper/meshes/arg/inner_knuckle_coarse.STL" />
       </geometry>
     </collision>
@@ -399,19 +399,19 @@
       <geometry>
         <mesh
-          filename="package://robowflex_resources/robotiq/85_gripper/meshes/arg/inner_finger_fine.STL" />
-      </geometry>
-      <material
-        name="">
-        <color
-          rgba="0.1 0.1 0.1 1" />
-      </material>
-    </visual>
-    <collision>
-      <origin
-        xyz="0 0 0"
-        rpy="0 0 0" />
-      <geometry>
-        <mesh
-          filename="package://robowflex_resources/robotiq/85_gripper/meshes/arg/inner_finger_coarse.STL" />
+          filename="package://moveit_benchmark_suite_resources/robots/robotiq/85_gripper/meshes/arg/inner_finger_fine.STL" />
+      </geometry>
+      <material
+        name="">
+        <color
+          rgba="0.1 0.1 0.1 1" />
+      </material>
+    </visual>
+    <collision>
+      <origin
+        xyz="0 0 0"
+        rpy="0 0 0" />
+      <geometry>
+        <mesh
+          filename="package://moveit_benchmark_suite_resources/robots/robotiq/85_gripper/meshes/arg/inner_finger_coarse.STL" />
       </geometry>
     </collision>
@@ -461,19 +461,19 @@
       <geometry>
         <mesh
-          filename="package://robowflex_resources/robotiq/85_gripper/meshes/arg/outer_knuckle_fine.STL" />
-      </geometry>
-      <material
-        name="">
-        <color
-          rgba="0.1 0.1 0.1 1" />
-      </material>
-    </visual>
-    <collision>
-      <origin
-        xyz="0 0 0"
-        rpy="0 0 0" />
-      <geometry>
-        <mesh
-          filename="package://robowflex_resources/robotiq/85_gripper/meshes/arg/outer_knuckle_coarse.STL" />
+          filename="package://moveit_benchmark_suite_resources/robots/robotiq/85_gripper/meshes/arg/outer_knuckle_fine.STL" />
+      </geometry>
+      <material
+        name="">
+        <color
+          rgba="0.1 0.1 0.1 1" />
+      </material>
+    </visual>
+    <collision>
+      <origin
+        xyz="0 0 0"
+        rpy="0 0 0" />
+      <geometry>
+        <mesh
+          filename="package://moveit_benchmark_suite_resources/robots/robotiq/85_gripper/meshes/arg/outer_knuckle_coarse.STL" />
       </geometry>
     </collision>
@@ -514,19 +514,19 @@
       <geometry>
         <mesh
-          filename="package://robowflex_resources/robotiq/85_gripper/meshes/arg/outer_finger_fine.STL" />
-      </geometry>
-      <material
-        name="">
-        <color
-          rgba="0.1 0.1 0.1 1" />
-      </material>
-    </visual>
-    <collision>
-      <origin
-        xyz="0 0 0"
-        rpy="0 0 0" />
-      <geometry>
-        <mesh
-          filename="package://robowflex_resources/robotiq/85_gripper/meshes/arg/outer_finger_coarse.STL" />
+          filename="package://moveit_benchmark_suite_resources/robots/robotiq/85_gripper/meshes/arg/outer_finger_fine.STL" />
+      </geometry>
+      <material
+        name="">
+        <color
+          rgba="0.1 0.1 0.1 1" />
+      </material>
+    </visual>
+    <collision>
+      <origin
+        xyz="0 0 0"
+        rpy="0 0 0" />
+      <geometry>
+        <mesh
+          filename="package://moveit_benchmark_suite_resources/robots/robotiq/85_gripper/meshes/arg/outer_finger_coarse.STL" />
       </geometry>
     </collision>

File: resources/robots/robotiq/force_torque_sensor/urdf/robotiq_fts300.urdf.xacro (robot description, xacro)
@@ -18,5 +18,5 @@
                 <origin xyz="0 0 0" rpy="0 0 0" />
                 <geometry>
-                    <mesh filename="package://robowflex_resources/robotiq/force_torque_sensor/meshes/visual/robotiq_fts300.stl"/>
+                    <mesh filename="package://moveit_benchmark_suite_resources/robots/robotiq/force_torque_sensor/meshes/visual/robotiq_fts300.stl"/>
                 </geometry>
                 <material name="black"/>
@@ -25,5 +25,5 @@
                 <origin xyz="0 0 0" rpy="0 0 0" />
                 <geometry>
-                    <mesh filename="package://robowflex_resources/robotiq/force_torque_sensor/meshes/collision/robotiq_fts300.stl"/>
+                    <mesh filename="package://moveit_benchmark_suite_resources/robots/robotiq/force_torque_sensor/meshes/collision/robotiq_fts300.stl"/>
                 </geometry>
             </collision>
