Commit message: Fix package path resolution

File: resources/robots/ur5/urdf/ur5.urdf.xacro (robot description, xacro)
@@ -73,13 +73,13 @@
       <visual>
         <geometry>
-          <mesh filename="package://robowflex_resources/ur/meshes/ur5/visual/base.dae" />
-        </geometry>
-        <material name="LightGrey">
-          <color rgba="0.7 0.7 0.7 1.0"/>
-        </material>
-      </visual>
-      <collision>
-        <geometry>
-          <mesh filename="package://robowflex_resources/ur/meshes/ur5/collision/base.stl" />
+          <mesh filename="package://moveit_benchmark_suite_resources/robots/ur5/meshes/ur5/visual/base.dae" />
+        </geometry>
+        <material name="LightGrey">
+          <color rgba="0.7 0.7 0.7 1.0"/>
+        </material>
+      </visual>
+      <collision>
+        <geometry>
+          <mesh filename="package://moveit_benchmark_suite_resources/robots/ur5/meshes/ur5/collision/base.stl" />
         </geometry>
       </collision>
@@ -104,13 +104,13 @@
       <visual>
         <geometry>
-          <mesh filename="package://robowflex_resources/ur/meshes/ur5/visual/shoulder.dae" />
-        </geometry>
-        <material name="LightGrey">
-          <color rgba="0.7 0.7 0.7 1.0"/>
-        </material>
-      </visual>
-      <collision>
-        <geometry>
-          <mesh filename="package://robowflex_resources/ur/meshes/ur5/collision/shoulder.stl" />
+          <mesh filename="package://moveit_benchmark_suite_resources/robots/ur5/meshes/ur5/visual/shoulder.dae" />
+        </geometry>
+        <material name="LightGrey">
+          <color rgba="0.7 0.7 0.7 1.0"/>
+        </material>
+      </visual>
+      <collision>
+        <geometry>
+          <mesh filename="package://moveit_benchmark_suite_resources/robots/ur5/meshes/ur5/collision/shoulder.stl" />
         </geometry>
       </collision>
@@ -136,13 +136,13 @@
       <visual>
         <geometry>
-          <mesh filename="package://robowflex_resources/ur/meshes/ur5/visual/upperarm.dae" />
-        </geometry>
-        <material name="LightGrey">
-          <color rgba="0.7 0.7 0.7 1.0"/>
-        </material>
-      </visual>
-      <collision>
-        <geometry>
-          <mesh filename="package://robowflex_resources/ur/meshes/ur5/collision/upperarm.stl" />
+          <mesh filename="package://moveit_benchmark_suite_resources/robots/ur5/meshes/ur5/visual/upperarm.dae" />
+        </geometry>
+        <material name="LightGrey">
+          <color rgba="0.7 0.7 0.7 1.0"/>
+        </material>
+      </visual>
+      <collision>
+        <geometry>
+          <mesh filename="package://moveit_benchmark_suite_resources/robots/ur5/meshes/ur5/collision/upperarm.stl" />
         </geometry>
       </collision>
@@ -167,13 +167,13 @@
       <visual>
         <geometry>
-          <mesh filename="package://robowflex_resources/ur/meshes/ur5/visual/forearm.dae" />
-        </geometry>
-        <material name="LightGrey">
-          <color rgba="0.7 0.7 0.7 1.0"/>
-        </material>
-      </visual>
-      <collision>
-        <geometry>
-          <mesh filename="package://robowflex_resources/ur/meshes/ur5/collision/forearm.stl" />
+          <mesh filename="package://moveit_benchmark_suite_resources/robots/ur5/meshes/ur5/visual/forearm.dae" />
+        </geometry>
+        <material name="LightGrey">
+          <color rgba="0.7 0.7 0.7 1.0"/>
+        </material>
+      </visual>
+      <collision>
+        <geometry>
+          <mesh filename="package://moveit_benchmark_suite_resources/robots/ur5/meshes/ur5/collision/forearm.stl" />
         </geometry>
       </collision>
@@ -198,13 +198,13 @@
       <visual>
         <geometry>
-          <mesh filename="package://robowflex_resources/ur/meshes/ur5/visual/wrist1.dae" />
-        </geometry>
-        <material name="LightGrey">
-          <color rgba="0.7 0.7 0.7 1.0"/>
-        </material>
-      </visual>
-      <collision>
-        <geometry>
-          <mesh filename="package://robowflex_resources/ur/meshes/ur5/collision/wrist1.stl" />
+          <mesh filename="package://moveit_benchmark_suite_resources/robots/ur5/meshes/ur5/visual/wrist1.dae" />
+        </geometry>
+        <material name="LightGrey">
+          <color rgba="0.7 0.7 0.7 1.0"/>
+        </material>
+      </visual>
+      <collision>
+        <geometry>
+          <mesh filename="package://moveit_benchmark_suite_resources/robots/ur5/meshes/ur5/collision/wrist1.stl" />
         </geometry>
       </collision>
@@ -229,13 +229,13 @@
       <visual>
         <geometry>
-          <mesh filename="package://robowflex_resources/ur/meshes/ur5/visual/wrist2.dae" />
-        </geometry>
-        <material name="LightGrey">
-          <color rgba="0.7 0.7 0.7 1.0"/>
-        </material>
-      </visual>
-      <collision>
-        <geometry>
-          <mesh filename="package://robowflex_resources/ur/meshes/ur5/collision/wrist2.stl" />
+          <mesh filename="package://moveit_benchmark_suite_resources/robots/ur5/meshes/ur5/visual/wrist2.dae" />
+        </geometry>
+        <material name="LightGrey">
+          <color rgba="0.7 0.7 0.7 1.0"/>
+        </material>
+      </visual>
+      <collision>
+        <geometry>
+          <mesh filename="package://moveit_benchmark_suite_resources/robots/ur5/meshes/ur5/collision/wrist2.stl" />
         </geometry>
       </collision>
@@ -260,13 +260,13 @@
       <visual>
         <geometry>
-          <mesh filename="package://robowflex_resources/ur/meshes/ur5/visual/wrist3.dae" />
-        </geometry>
-        <material name="LightGrey">
-          <color rgba="0.7 0.7 0.7 1.0"/>
-        </material>
-      </visual>
-      <collision>
-        <geometry>
-          <mesh filename="package://robowflex_resources/ur/meshes/ur5/collision/wrist3.stl" />
+          <mesh filename="package://moveit_benchmark_suite_resources/robots/ur5/meshes/ur5/visual/wrist3.dae" />
+        </geometry>
+        <material name="LightGrey">
+          <color rgba="0.7 0.7 0.7 1.0"/>
+        </material>
+      </visual>
+      <collision>
+        <geometry>
+          <mesh filename="package://moveit_benchmark_suite_resources/robots/ur5/meshes/ur5/collision/wrist3.stl" />
         </geometry>
       </collision>

File: resources/robots/ur5/urdf/ur5_robotiq85.urdf.xacro (robot description, xacro)
@@ -3,7 +3,7 @@
        name="ur5_robotiq85" >
   <!-- common stuff -->
-  <xacro:include filename="$(find robowflex_resources)/ur/robots/common.gazebo.xacro" />
+  <xacro:include filename="$(find moveit_benchmark_suite_resources)/robots/ur5/urdf/common.gazebo.xacro" />
   <!-- ur5 -->
-  <xacro:include filename="$(find robowflex_resources)/ur/robots/ur5.urdf.xacro" />
+  <xacro:include filename="$(find moveit_benchmark_suite_resources)/robots/ur5/urdf/ur5.urdf.xacro" />
   <!-- arm -->
   <xacro:ur5_robot prefix=""/>
@@ -16,5 +16,5 @@
  </joint>
  <!-- Force Torque Sensor -->
- <xacro:include filename="$(find robowflex_resources)/robotiq/force_torque_sensor/urdf/robotiq_fts300.urdf.xacro" />
+ <xacro:include filename="$(find moveit_benchmark_suite_resources)/robots/robotiq/force_torque_sensor/urdf/robotiq_fts300.urdf.xacro" />
  <xacro:robotiq_fts300 prefix="" parent="ee_link" >
    <origin xyz="0.035 0 0.0" rpy="0.0 0 -1.57"/>
@@ -22,5 +22,5 @@
  <!-- GRIPPER -->
  <!-- Import robotiq gazebo and gripper description -->
- <xacro:include filename="$(find robowflex_resources)/robotiq/85_gripper/urdf/robotiq_85_gripper.urdf.xacro" />
+ <xacro:include filename="$(find moveit_benchmark_suite_resources)/robots/robotiq/85_gripper/urdf/robotiq_85_gripper.urdf.xacro" />
  <xacro:robotiq_85_gripper prefix="" parent="fts_toolside" >
    <origin xyz="0.0 0.0 -0.037" rpy="0.0 0.0 1.57"/>
