Commit message: Add fixed frame transform attribute for scenes

File: resources/scenes/bbt/panda/mesh_16k.urdf.xacro (robot description, xacro)
@@ -3,17 +3,24 @@
   <xacro:include filename="$(find urdf_to_scene)/config/utils.xacro" />
   <xacro:include filename="$(find moveit_benchmark_suite_resources)/objects/metadata.xacro" />
-  <link name="world" />
+  <!-- Transform World to Robot -->
+  <link name="world"/>
+  <planning_fft name="panda_link0"
+                parent="world"
+                xyz="0.365 0 0"/>
+  <!-- World -->
   <xacro:framemesh name="boxlid"
-                       frame_id="world"
-                       xyz="${0.16 + boxlid['bb'][1]/2} ${-boxlid['bb'][2]/2} ${boxlid['bb'][0]/2}" rpy="0 ${pi/2} ${pi/2}"
-                       metadata="${boxlid}"/>
+                   frame_id="world"
+                   xyz="0 ${-boxlid['bb'][2]/2} ${boxlid['bb'][0]/2}"
+                   rpy="0 ${pi/2} ${pi/2}"
+                   metadata="${boxlid}"/>
   <xacro:framemesh name="clearbox1"
-                       frame_id="world"
-                       xyz="${0.16 + clearbox['bb'][1]/2} ${-(clearbox['bb'][0]/2 + boxlid['bb'][2]/2)} 0" rpy="0 0 ${pi/2}"
-                       metadata="${clearbox}"/>
+                   frame_id="world"
+                   xyz="0 ${-(clearbox['bb'][0]/2 + boxlid['bb'][2]/2)} 0"
+                   rpy="0 0 ${pi/2}"
+                   metadata="${clearbox}"/>
   <xacro:framemesh name="clearbox2"
-                       frame_id="clearbox1"
-                       xyz="${clearbox['bb'][0] + boxlid['bb'][2]} 0 0" rpy="0 0 0"
-                       metadata="${clearbox}"/>
+                   frame_id="clearbox1"
+                   xyz="${clearbox['bb'][0] + boxlid['bb'][2]} 0 0" rpy="0 0 0"
+                   metadata="${clearbox}"/>
   <xacro:macro name="linearpattern" params="current:=0 frame_id:=^ index:=0 until:=^ xyz:=^ rpy=^|'0 0 0' gap:=^">
     <xacro:if value="${until > current}">

File: resources/scenes/bbt/panda/primitive.urdf.xacro (robot description, xacro)
@@ -4,31 +4,35 @@
   <xacro:include filename="$(find urdf_to_scene)/config/opencrate.urdf.xacro" />
   <xacro:include filename="$(find moveit_benchmark_suite_resources)/objects/metadata.xacro" />
-  <link name="world" />
+  <!-- Transform World to Robot -->
+  <link name="world"/>
+  <planning_fft name="panda_link0"
+                parent="world"
+                xyz="0.365 0 0"/>
+  <!-- World -->
   <xacro:framebox name="boxlid"
-                  frame_id="world"
                   dimensions="${boxlid['bb'][1]} ${boxlid['bb'][2]} ${boxlid['bb'][0]}"
-                  xyz="${0.16 + boxlid['bb'][1]/2} 0 0"/>
+                  frame_id="world"/>
   <xacro:opencrate name="clearbox1"
-                   frame_id="world"
-                   xyz="${0.16 + clearbox['bb'][1]/2} ${-(clearbox['bb'][0]/2 + boxlid['bb'][2]/2)} 0" rpy="0 0 0"
+                   frame_id="boxlid"
+                   xyz="0 ${-(clearbox['bb'][0]/2 + boxlid['bb'][2]/2)} ${-boxlid['bb'][0]}"
                    dimensions="${clearbox['bb'][1]} ${clearbox['bb'][0]} ${clearbox['bb'][2]}"
                    thickness="${clearbox['subframes']['stack']['xyz'][2]}"/>
   <xacro:opencrate name="clearbox2"
                    frame_id="clearbox1"
-                   xyz="0 ${clearbox['bb'][0] + boxlid['bb'][2]} 0" rpy="0 0 0"
+                   xyz="0 ${clearbox['bb'][0] + boxlid['bb'][2]} 0"
                    dimensions="${clearbox['bb'][1]} ${clearbox['bb'][0]} ${clearbox['bb'][2]}"
                    thickness="0.00709"/>
   <xacro:macro name="linearpattern" params="current:=0 frame_id:=^ index:=0 until:=^ xyz:=^ rpy=^|'0 0 0' gap:=^">
     <xacro:if value="${until > current}">
-      <xacro:framebox name="woodblock${index+current}"
-                      frame_id="${frame_id}"
-                      dimensions="${woodblock['bb'][0]} ${woodblock['bb'][1]} ${woodblock['bb'][2]}"
-                      xyz="${float(xyz.split()[0]) + current*float(gap.split()[0])}
-                           ${float(xyz.split()[1]) + current*float(gap.split()[1])}
-                           ${float(xyz.split()[2]) + current*float(gap.split()[2])}" />
-      <xacro:linearpattern current="${current+1}" index="${index}"/>
+        <xacro:framebox name="woodblock${index+current}"
+                        frame_id="${frame_id}"
+                        dimensions="${woodblock['bb'][0]} ${woodblock['bb'][1]} ${woodblock['bb'][2]}"
+                        xyz="${float(xyz.split()[0]) + current*float(gap.split()[0])}
+                             ${float(xyz.split()[1]) + current*float(gap.split()[1])}
+                             ${float(xyz.split()[2]) + current*float(gap.split()[2])}" />
+        <xacro:linearpattern current="${current+1}" index="${index}"/>
     </xacro:if>
   </xacro:macro>
-  <xacro:linearpattern index="1"  until="4"  frame_id="clearbox1"  gap="0 ${woodblock['bb'][1]*2} 0" xyz="${3*woodblock['bb'][0]} ${(-3*woodblock['bb'][0])} 0" rpy="0 0 0"/>
+  <xacro:linearpattern index="1"  until="4"  frame_id="clearbox1" gap="0 ${woodblock['bb'][1]*2} 0" xyz="${3*woodblock['bb'][0]} ${(-3*woodblock['bb'][0])} 0" rpy="0 0 0"/>
   <xacro:linearpattern index="5"  until="4"  frame_id="woodblock1/bottom" gap="0 ${woodblock['bb'][1]*2} 0" xyz="${-2*woodblock['bb'][0]} 0 0"/>
   <xacro:linearpattern index="9"  until="4"  frame_id="woodblock5/bottom" gap="0 ${woodblock['bb'][1]*2} 0" xyz="${-2*woodblock['bb'][0]} 0 0"/>
