Commit message: Fix urdf warning

File: resources/robots/robotiq/force_torque_sensor/urdf/robotiq_fts300.urdf.xacro (robot description, xacro)
@@ -20,5 +20,7 @@
                     <mesh filename="package://moveit_benchmark_suite_resources/robots/robotiq/force_torque_sensor/meshes/visual/robotiq_fts300.stl"/>
                 </geometry>
-                <material name="black"/>
+                <material name="black">
+                    <color rgba="0 0 0 1.0"/>
+                </material>
             </visual>
             <collision>
