Commit message: Fix mesh path

File: resources/robots/ur5/urdf/ur5.urdf.xacro (robot description, xacro)
@@ -73,13 +73,13 @@
       <visual>
         <geometry>
-          <mesh filename="package://moveit_benchmark_suite_resources/robots/ur5/meshes/ur5/visual/base.dae" />
-        </geometry>
-        <material name="LightGrey">
-          <color rgba="0.7 0.7 0.7 1.0"/>
-        </material>
-      </visual>
-      <collision>
-        <geometry>
-          <mesh filename="package://moveit_benchmark_suite_resources/robots/ur5/meshes/ur5/collision/base.stl" />
+          <mesh filename="package://moveit_benchmark_suite_resources/robots/ur5/meshes/visual/base.dae" />
+        </geometry>
+        <material name="LightGrey">
+          <color rgba="0.7 0.7 0.7 1.0"/>
+        </material>
+      </visual>
+      <collision>
+        <geometry>
+          <mesh filename="package://moveit_benchmark_suite_resources/robots/ur5/meshes/collision/base.stl" />
         </geometry>
       </collision>
@@ -104,13 +104,13 @@
       <visual>
         <geometry>
-          <mesh filename="package://moveit_benchmark_suite_resources/robots/ur5/meshes/ur5/visual/shoulder.dae" />
-        </geometry>
-        <material name="LightGrey">
-          <color rgba="0.7 0.7 0.7 1.0"/>
-        </material>
-      </visual>
-      <collision>
-        <geometry>
-          <mesh filename="package://moveit_benchmark_suite_resources/robots/ur5/meshes/ur5/collision/shoulder.stl" />
+          <mesh filename="package://moveit_benchmark_suite_resources/robots/ur5/meshes/visual/shoulder.dae" />
+        </geometry>
+        <material name="LightGrey">
+          <color rgba="0.7 0.7 0.7 1.0"/>
+        </material>
+      </visual>
+      <collision>
+        <geometry>
+          <mesh filename="package://moveit_benchmark_suite_resources/robots/ur5/meshes/collision/shoulder.stl" />
         </geometry>
       </collision>
@@ -136,13 +136,13 @@
       <visual>
         <geometry>
-          <mesh filename="package://moveit_benchmark_suite_resources/robots/ur5/meshes/ur5/visual/upperarm.dae" />
-        </geometry>
-        <material name="LightGrey">
-          <color rgba="0.7 0.7 0.7 1.0"/>
-        </material>
-      </visual>
-      <collision>
-        <geometry>
-          <mesh filename="package://moveit_benchmark_suite_resources/robots/ur5/meshes/ur5/collision/upperarm.stl" />
+          <mesh filename="package://moveit_benchmark_suite_resources/robots/ur5/meshes/visual/upperarm.dae" />
+        </geometry>
+        <material name="LightGrey">
+          <color rgba="0.7 0.7 0.7 1.0"/>
+        </material>
+      </visual>
+      <collision>
+        <geometry>
+          <mesh filename="package://moveit_benchmark_suite_resources/robots/ur5/meshes/collision/upperarm.stl" />
         </geometry>
       </collision>
@@ -167,13 +167,13 @@
       <visual>
         <geometry>
-          <mesh filename="package://moveit_benchmark_suite_resources/robots/ur5/meshes/ur5/visual/forearm.dae" />
-        </geometry>
-        <material name="LightGrey">
-          <color rgba="0.7 0.7 0.7 1.0"/>
-        </material>
-      </visual>
-      <collision>
-        <geometry>
-          <mesh filename="package://moveit_benchmark_suite_resources/robots/ur5/meshes/ur5/collision/forearm.stl" />
+          <mesh filename="package://moveit_benchmark_suite_resources/robots/ur5/meshes/visual/forearm.dae" />
+        </geometry>
+        <material name="LightGrey">
+          <color rgba="0.7 0.7 0.7 1.0"/>
+        </material>
+      </visual>
+      <collision>
+        <geometry>
+          <mesh filename="package://moveit_benchmark_suite_resources/robots/ur5/meshes/collision/forearm.stl" />
         </geometry>
       </collision>
@@ -198,13 +198,13 @@
       <visual>
         <geometry>
-          <mesh filename="package://moveit_benchmark_suite_resources/robots/ur5/meshes/ur5/visual/wrist1.dae" />
-        </geometry>
-        <material name="LightGrey">
-          <color rgba="0.7 0.7 0.7 1.0"/>
-        </material>
-      </visual>
-      <collision>
-        <geometry>
-          <mesh filename="package://moveit_benchmark_suite_resources/robots/ur5/meshes/ur5/collision/wrist1.stl" />
+          <mesh filename="package://moveit_benchmark_suite_resources/robots/ur5/meshes/visual/wrist1.dae" />
+        </geometry>
+        <material name="LightGrey">
+          <color rgba="0.7 0.7 0.7 1.0"/>
+        </material>
+      </visual>
+      <collision>
+        <geometry>
+          <mesh filename="package://moveit_benchmark_suite_resources/robots/ur5/meshes/collision/wrist1.stl" />
         </geometry>
       </collision>
@@ -229,13 +229,13 @@
       <visual>
         <geometry>
-          <mesh filename="package://moveit_benchmark_suite_resources/robots/ur5/meshes/ur5/visual/wrist2.dae" />
-        </geometry>
-        <material name="LightGrey">
-          <color rgba="0.7 0.7 0.7 1.0"/>
-        </material>
-      </visual>
-      <collision>
-        <geometry>
-          <mesh filename="package://moveit_benchmark_suite_resources/robots/ur5/meshes/ur5/collision/wrist2.stl" />
+          <mesh filename="package://moveit_benchmark_suite_resources/robots/ur5/meshes/visual/wrist2.dae" />
+        </geometry>
+        <material name="LightGrey">
+          <color rgba="0.7 0.7 0.7 1.0"/>
+        </material>
+      </visual>
+      <collision>
+        <geometry>
+          <mesh filename="package://moveit_benchmark_suite_resources/robots/ur5/meshes/collision/wrist2.stl" />
         </geometry>
       </collision>
@@ -260,13 +260,13 @@
       <visual>
         <geometry>
-          <mesh filename="package://moveit_benchmark_suite_resources/robots/ur5/meshes/ur5/visual/wrist3.dae" />
-        </geometry>
-        <material name="LightGrey">
-          <color rgba="0.7 0.7 0.7 1.0"/>
-        </material>
-      </visual>
-      <collision>
-        <geometry>
-          <mesh filename="package://moveit_benchmark_suite_resources/robots/ur5/meshes/ur5/collision/wrist3.stl" />
+          <mesh filename="package://moveit_benchmark_suite_resources/robots/ur5/meshes/visual/wrist3.dae" />
+        </geometry>
+        <material name="LightGrey">
+          <color rgba="0.7 0.7 0.7 1.0"/>
+        </material>
+      </visual>
+      <collision>
+        <geometry>
+          <mesh filename="package://moveit_benchmark_suite_resources/robots/ur5/meshes/collision/wrist3.stl" />
         </geometry>
       </collision>
