Commit message: Remove redefinition of pi in xacro

File: resources/robots/robotiq/85_gripper/urdf/robotiq_85_gripper.urdf.xacro (robot description, xacro)
@@ -2,5 +2,4 @@
 <robot name="robotiq_85_gripper" xmlns:xacro="http://ros.org/wiki/xacro">
 	<xacro:include filename="$(find moveit_benchmark_suite_resources)/robots/robotiq/85_gripper/urdf/robotiq_85_gripper.transmission.xacro" />
-	<xacro:property name="pi" value="3.14159"/>
 	<xacro:macro name="mimic_joint_plugin_gazebo" params="name_prefix parent_joint mimic_joint has_pid:=false multiplier:=1.0 offset:=0 sensitiveness:=0.0 max_effort:=1.0 robot_namespace:=''">
 		<gazebo>

File: resources/robots/robotiq/85_gripper/urdf/robotiq_arg85_description.urdf.xacro (robot description, xacro)
@@ -3,5 +3,4 @@
   name="robotiq_85_gripper"  xmlns:xacro="http://ros.org/wiki/xacro">
   <xacro:include filename="$(find moveit_benchmark_suite_resources)/robots/robotiq/85_gripper/urdf/robotiq_85_gripper.transmission.xacro" />
-	<xacro:property name="pi" value="3.14159"/>
   <xacro:macro name="robotiq_85_gripper" params="prefix parent *origin">
   <joint name="${prefix}robotiq_85_base_joint" type="fixed">

File: resources/robots/ur5/urdf/ur5.urdf.xacro (robot description, xacro)
@@ -3,5 +3,4 @@
   <xacro:include filename="ur.transmission.xacro" />
   <xacro:include filename="ur.gazebo.xacro" />
-  <xacro:property name="pi" value="3.14159265" />
   <!-- Inertia parameters -->
   <xacro:property name="base_mass" value="4.0" />  <!-- This mass might be incorrect -->
